File: kicad/qx10_titan_memory/qx10_titan_memory.kicad_pcb (KiCad board)
At the start: 2 copper layers, 0 parts

Commit message: kicad: Initial board layout for titan memory board
Parts:
- added C1: Filter Cap, Capacitor_THT:CP_Radial_D5.0mm_P2.50mm, F.Cu at (95.7, 132.1)
- added J1: QX-PC Connector, Connector_PinHeader_2.54mm:PinHeader_2x20_P2.54mm_Vertical, F.Cu at (62.5, 81.8)
- added R1: 100, Resistor_THT:R_Axial_DIN0207_L6.3mm_D2.5mm_P10.16mm_Horizontal, F.Cu at (72.1, 99.1)
- added R2: 10, Resistor_THT:R_Axial_DIN0207_L6.3mm_D2.5mm_P10.16mm_Horizontal, F.Cu at (91.2, 95.5)
- added RN1: 100, Resistor_THT:R_Array_SIP8, F.Cu at (71.4, 110.2)
- added RN2: 100, Resistor_THT:R_Array_SIP8, F.Cu at (71.4, 114.3)
- added RN3: 100, Resistor_THT:R_Array_SIP8, F.Cu at (71.4, 126.7)
- added U1: 74LS244, Package_DIP:DIP-20_W7.62mm_Socket, F.Cu at (77.0, 81.8)
- added U10: MT4264, Package_DIP:DIP-16_W7.62mm_Socket, F.Cu at (100.8, 112.5)
- added U11: MT4264, Package_DIP:DIP-16_W7.62mm_Socket, F.Cu at (113.8, 112.5)
- added U12: MT4264, Package_DIP:DIP-16_W7.62mm_Socket, F.Cu at (126.7, 112.5)
- added U13: MT4264, Package_DIP:DIP-16_W7.62mm_Socket, F.Cu at (139.7, 112.5)
- added U14: MT4264, Package_DIP:DIP-16_W7.62mm_Socket, F.Cu at (152.6, 112.5)
- added U15: MT4264, Package_DIP:DIP-16_W7.62mm_Socket, F.Cu at (165.5, 112.5)
- added U16: MT4264, Package_DIP:DIP-16_W7.62mm_Socket, F.Cu at (178.5, 112.5)
- added U17: MT4264, Package_DIP:DIP-16_W7.62mm_Socket, F.Cu at (191.4, 112.5)
- added U18: MT4264, Package_DIP:DIP-16_W7.62mm_Socket, F.Cu at (204.3, 112.5)
- added U19: MT4264, Package_DIP:DIP-16_W7.62mm_Socket, F.Cu at (217.3, 112.5)
- added U2: MT4264, Package_DIP:DIP-16_W7.62mm_Socket, F.Cu at (100.8, 81.8)
- added U20: MT4264, Package_DIP:DIP-16_W7.62mm_Socket, F.Cu at (230.2, 112.5)
- added U21: MT4264, Package_DIP:DIP-16_W7.62mm_Socket, F.Cu at (243.2, 112.5)
- added U22: MT4264, Package_DIP:DIP-16_W7.62mm_Socket, F.Cu at (256.1, 112.5)
- added U23: MT4264, Package_DIP:DIP-16_W7.62mm_Socket, F.Cu at (269.0, 112.5)
- added U24: MT4264, Package_DIP:DIP-16_W7.62mm_Socket, F.Cu at (282.0, 112.5)
- added U25: MT4264, Package_DIP:DIP-16_W7.62mm_Socket, F.Cu at (294.9, 112.5)
- added U26: MT4264, Package_DIP:DIP-16_W7.62mm_Socket, F.Cu at (204.3, 81.8)
- added U27: MT4264, Package_DIP:DIP-16_W7.62mm_Socket, F.Cu at (217.3, 81.8)
- added U28: MT4264, Package_DIP:DIP-16_W7.62mm_Socket, F.Cu at (230.2, 81.8)
- added U29: MT4264, Package_DIP:DIP-16_W7.62mm_Socket, F.Cu at (243.2, 81.8)
- added U3: MT4264, Package_DIP:DIP-16_W7.62mm_Socket, F.Cu at (113.8, 81.8)
- added U30: MT4264, Package_DIP:DIP-16_W7.62mm_Socket, F.Cu at (256.1, 81.8)
- added U31: MT4264, Package_DIP:DIP-16_W7.62mm_Socket, F.Cu at (269.0, 81.8)
- added U32: MT4264, Package_DIP:DIP-16_W7.62mm_Socket, F.Cu at (282.0, 81.8)
- added U33: MT4264, Package_DIP:DIP-16_W7.62mm_Socket, F.Cu at (294.9, 81.8)
- added U4: MT4264, Package_DIP:DIP-16_W7.62mm_Socket, F.Cu at (126.7, 81.8)
- added U5: MT4264, Package_DIP:DIP-16_W7.62mm_Socket, F.Cu at (139.7, 81.8)
- added U6: MT4264, Package_DIP:DIP-16_W7.62mm_Socket, F.Cu at (152.6, 81.8)
- added U7: MT4264, Package_DIP:DIP-16_W7.62mm_Socket, F.Cu at (165.5, 81.8)
- added U8: MT4264, Package_DIP:DIP-16_W7.62mm_Socket, F.Cu at (178.5, 81.8)
- added U9: MT4264, Package_DIP:DIP-16_W7.62mm_Socket, F.Cu at (191.4, 81.8)
Other:
- board outline added: 254 x 63.5 mm
- board text added: "BANK0"
- board text added: "BANK1"
- board text added: "BANK2"
- board text added: "BANK3"
