File: kicad/qx10_titan_memory/qx10_titan_memory.kicad_sch (KiCad schematic)
At the start: 40 parts, among them J1 QX-PC Connector, U1 74LS244, U10 MT4264, U11 MT4264, U12 MT4264, U13 MT4264, U14 MT4264, U15 MT4264, U16 MT4264, U17 MT4264, U18 MT4264, U19 MT4264, U2 MT4264, U20 MT4264, U21 MT4264, U22 MT4264, U23 MT4264, U24 MT4264, U25 MT4264, U26 MT4264, U27 MT4264, U28 MT4264, U29 MT4264, U3 MT4264, U30 MT4264, U31 MT4264, U32 MT4264, U33 MT4264, U4 MT4264, U5 MT4264, U6 MT4264, U7 MT4264, U8 MT4264, U9 MT4264

Commit message: kicad: Initial board layout for titan memory board
Parts:
- C1: footprint (none) -> Capacitor_THT:CP_Radial_D5.0mm_P2.50mm
- J1: footprint (none) -> Connector_PinHeader_2.54mm:PinHeader_2x20_P2.54mm_Vertical
- R1, R2: footprint (none) -> Resistor_THT:R_Axial_DIN0207_L6.3mm_D2.5mm_P10.16mm_Horizontal
- U1: footprint (none) -> Package_DIP:DIP-20_W7.62mm_Socket
- U10, U11, U12, U13, U14, U15, U16, U17, U18, U19, U2, U20, U21, U22, U23, U24, U25, U26, U27, U28, U29, U3, U30, U31, U32, U33, U4, U5, U6, U7, U8, U9: footprint (none) -> Package_DIP:DIP-16_W7.62mm_Socket
