File: kicad/qx10_titan_qxpc/qx10_titan_qxpc.kicad_sch (KiCad schematic)
At the start: 31 parts, among them CN1 Edge Connector, J2 Memory Board Header, U1 74LS244, U10 74LS21, U11 74LS74, U12 74LS74, U13 74F74, U14 74LS244, U15 74LS373, U16 74LS373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

Commit message: kicad: Add some notes to titan qxpc schematic
Other:
- note added: "INTL - 8088 Access IO Port 0x400 INTH1 - 8088 Access VRAM (0xB0000-0xBFFFF) INTH2 - 8088 Access IO Port Besides 0x400"
- note added: "Port D1 (Read) - IO/Mem Transfer"
- note added: "Port D1 (Write) - IO/Mem Transfer"
- note added: "Port D3 (Read) - Low Address Byte"
- note added: "Port D5 (Read) - High Address Byte"
- note added: "Port D7 (Write)- Trigger 8088 IRQ"
- moved on the sheet: R2, U10B, U11A, U13A, U13B, U14, U15, U16, U17, U18, U19, U6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

Commit message: kicad: Add a few more notes to titan qxpc schematic
Other:
- note added: "Port D1 - OE2 Port D3 - OE4 Port D5 - OE3 Port D7 - OE1"
Changed lines of the file:
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@@
+    (effects (font (size 1.27 1.27)) (justify left bottom))
+  )
+  (text "Port D1 - OE2\nPort D3 - OE4\nPort D5 - OE3\nPort D7 - OE1"
+    (at 31.0896 161.1884 0)
     (effects (font (size 1.27 1.27)) (justify left bottom))
   )
