File: kicad/memory_expansion/memory_expansion.kicad_sch (KiCad schematic)
At the start: 22 parts, among them CN1 QX10_Bus, U1 74LS541, U2 74LS541, U3 74LS245, U4 74LS541, U5 EPM7160SLC84-7, U6 AS6C4008-55PCN, U7 AS6C4008-55PCN

Commit message: kicad: update PLCC socket part numbers for memory expansion board
Parts:
- U5: Digikey 2057-PLCC-84-AT-ND -> 3M8411B1-ND; MFN PLCC-84-AT -> 8484-11B1-RK-TP; Mouser (none) -> 517-8484-11B1-RK-TP
Changed lines of the file:
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@@
       (effects (font (size 1.27 1.27)) (justify left bottom) hide)
     )
-    (property "MFN" "PLCC-84-AT" (id 4) (at 238.76 87.63 0)
+    (property "MFN" "8484-11B1-RK-TP" (id 4) (at 238.76 87.63 0)
       (effects (font (size 1.27 1.27)) hide)
     )
-    (property "Digikey" "2057-PLCC-84-AT-ND" (id 5) (at 238.76 87.63 0)
+    (property "Digikey" "3M8411B1-ND" (id 5) (at 238.76 87.63 0)
       (effects (font (size 1.27 1.27)) hide)
     )
+    (property "Mouser" "517-8484-11B1-RK-TP " (id 6) (at 238.76 87.63 0)
+      (effects (font (size 1.27 1.27)) hide)
+    )
