File: kicad/qx10_multifont/qx10_multifont.kicad_sch (KiCad schematic)
At the start: 44 parts, among them J1 Jumper_3_Open, J2 Jumper_3_Open, J3 Serial, U1 74LS245, U10 LS74, U12 74LS374, U13 74LS374, U16 MCP23S17, U17 74LS541, U2 74LS541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

Commit message: kicad: Update parts list for multifont card
Parts:
- J1, J2: Digikey (none) -> 609-3468-ND; MFR (none) -> 68001-103HLF
- J3: Digikey (none) -> 609-3271-ND; MFR (none) -> 68001-104HLF
- TP1, TP2, TP3, TP4, TP5, TP6, X1: now not fitted
- U16: Digikey (none) -> MCP23S17-E/SP-ND; MFR (none) -> MCP23S17-E/SP
- U27: Digikey (none) -> ATMEGA32A-PU-ND; MFR (none) -> ATMEGA32A-PU
Changed lines of the file:
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@@
 			)
 		)
-		(property "MFR" ""
+		(property "MFR" "MCP23S17-E/SP"
 			(at 351.79 347.98 0)
 			(effects
@@
 			)
 		)
-		(property "Digikey" ""
+		(property "Digikey" "MCP23S17-E/SP-ND"
 			(at 351.79 347.98 0)
 			(effects
@@
 			)
 		)
-		(property "MFR" ""
+		(property "MFR" "68001-103HLF"
 			(at 125.73 373.38 0)
 			(effects
@@
 			)
 		)
-		(property "Digikey" ""
+		(property "Digikey" "609-3468-ND"
 			(at 125.73 373.38 0)
 			(effects
@@
 			)
 		)
-		(property "MFR" ""
+		(property "MFR" "68001-103HLF"
 			(at 125.73 391.16 0)
 			(effects
@@
 			)
 		)
-		(property "Digikey" ""
+		(property "Digikey" "609-3468-ND"
 			(at 125.73 391.16 0)
 			(effects
@@
 		(in_bom yes)
 		(on_board yes)
-		(dnp no)
+		(dnp yes)
 		(property "Reference" "X1"
 			(at 24.13 351.79 0)
@@
 		(in_bom yes)
 		(on_board yes)
-		(dnp no)
+		(dnp yes)
 		(property "Reference" "X1"
 			(at 22.86 308.61 0)
@@
 		(in_bom yes)
 		(on_board yes)
-		(dnp no)
+		(dnp yes)
 		(property "Reference" "X1"
 			(at 26.6192 174.625 0)
@@
 		(in_bom yes)
 		(on_board yes)
-		(dnp no)
+		(dnp yes)
 		(property "Reference" "X1"
 			(at 23.4442 97.155 0)
@@
 		(in_bom yes)
 		(on_board yes)
-		(dnp no)
+		(dnp yes)
 		(property "Reference" "TP2"
 			(at 89.5985 156.21 90)
@@
 		(in_bom yes)
 		(on_board yes)
-		(dnp no)
+		(dnp yes)
 		(property "Reference" "TP4"
 			(at 109.9185 340.36 90)
@@
 		(in_bom yes)
 		(on_board yes)
-		(dnp no)
+		(dnp yes)
 		(property "Reference" "TP3"
 			(at 89.5985 158.75 90)
@@
 		(in_bom yes)
 		(on_board yes)
-		(dnp no)
+		(dnp yes)
 		(property "Reference" "TP5"
 			(at 73.66 156.9084 0)
@@
 			)
 		)
+		(property "Digikey" "609-3271-ND"
+			(at 241.3 252.73 90)
+			(effects
+				(font
+					(size 1.27 1.27)
+				)
+				(hide yes)
+			)
+		)
+		(property "MFR" "68001-104HLF "
+			(at 241.3 252.73 90)
+			(effects
+				(font
+					(size 1.27 1.27)
+				)
+				(hide yes)
+			)
+		)
 		(pin "4"
 		)
@@
 		(in_bom yes)
 		(on_board yes)
-		(dnp no)
+		(dnp yes)
 		(property "Reference" "TP1"
 			(at 89.5985 153.67 90)
@@
 		(in_bom yes)
 		(on_board yes)
-		(dnp no)
+		(dnp yes)
 		(property "Reference" "TP6"
 			(at 378.46 135.8899 90)
@@
 			)
 		)
-		(property "MFR" ""
+		(property "MFR" "ATMEGA32A-PU"
 			(at 303.53 220.98 0)
 			(effects
@@
 			)
 		)
-		(property "Digikey" ""
+		(property "Digikey" "ATMEGA32A-PU-ND"
 			(at 303.53 220.98 0)
 			(effects
