File: kicad/qx10_titan_clone/qx10_titan_clone.kicad_pcb (KiCad board)
At the start: 2 copper layers, 281 x 79 mm, 50 parts, among them CN1 Edge Connector, U1 74LS245, U10 74LS74, U11 74LS74, U12 74LS244, U13 74LS373, U14 74LS373, U15 GAL16V8, U16 74LS373, U17 74LS373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

Commit message: kicad: Route QXPC Clone PCB and update BOM
Parts:
- C21, C22: value 23pf -> 30pf
- R1, R2, R3: value 230 -> 220
- RN1: value R_Network07 -> 4.7k
- moved R3 31.1 mm to (273.1, 52.6), turned to 90 degrees
- moved C22 26.2 mm to (251.8, 32.5), turned to 0 degrees
- moved C21 17.1 mm to (262.0, 32.5), turned to 180 degrees
- moved Y1 13.3 mm to (259.3, 37.6), turned to 180 degrees
- moved C18 11.9 mm to (245.1, 46.2)
- moved U18 11.9 mm to (248.9, 51.3)
- renumbered REF** to H1, REF** to H2
Connections:
- U1 pad 1: /U2OE -> /~{RD}
- U6 pad 21: /A10 -> /Q10
- U6 pad 23: /A11 -> /Q11
- U6 pad 24: /A9 -> /Q9
- U6 pad 25: /A8 -> /Q8
Routing:
- net +5V: track 0.00 -> 900.5 mm, vias 0 -> 5
- net /~{RD}: track 0.00 -> 365.2 mm, vias 0 -> 4
- net /DIO5: track 0.00 -> 363.3 mm, vias 0 -> 6
- net /DIO6: track 0.00 -> 359.9 mm, vias 0 -> 5
- net /DIO7: track 0.00 -> 356.5 mm, vias 0 -> 3
- net /DIO4: track 0.00 -> 355.9 mm, vias 0 -> 6
- net /DIO0: track 0.00 -> 338.0 mm, vias 0 -> 3
- net /ALE: track 0.00 -> 335.5 mm, vias 0 -> 5
- net /DIO1: track 0.00 -> 333.2 mm, vias 0 -> 4
- net /DIO2: track 0.00 -> 333.2 mm, vias 0 -> 4
- net /A10: track 0.00 -> 324.2 mm, vias 0 -> 4
- net /DIO3: track 0.00 -> 320.1 mm, vias 0 -> 4
- net /A8: track 0.00 -> 312.7 mm, vias 0 -> 3
- net /A9: track 0.00 -> 306.7 mm, vias 0 -> 3
- net /~{WR}: track 0.00 -> 299.6 mm, vias 0 -> 4
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- added copper zone on B.Cu, net GND
Other:
- board text added: "V2 board"

Commit message: kicad: Update titan clone to kicad 9 and add BOM CSV
Routing:
- net /~{INTH2}: track 62.8 -> 63.4 mm
- net /~{INTH1}: track 75.0 -> 75.5 mm
