File: kicad/qx10_titan_clone/qx10_titan_clone.kicad_sch (KiCad schematic)
At the start: 48 parts, among them CN1 Edge Connector, U1 74LS245, U10 74LS74, U11 74LS74, U12 74LS244, U13 74LS373, U14 74LS373, U15 GAL16V8, U16 74LS373, U17 74LS373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

Commit message: kicad: Route QXPC Clone PCB and update BOM
Parts:
- C1, C10, C11, C12, C13, C14, C15, C16, C17, C18, C19, C2, C20, C3, C4, C5, C6, C7, C8, C9: MFR (none) -> RDER72A104K1S1H03A; Mouser (none) -> 81-RDER72A104K1S1H3A
- C21, C22: value 23pf -> 30pf; MFR (none) -> C315C300F3G5TA; Mouser (none) -> 80-C315C300F3G5TA
- R1, R2, R3: value 230 -> 220; MFR (none) -> CFR-25JR-52-220R; Mouser (none) -> 603-CFR-25JR-52220R
- RN1: value R_Network07 -> 4.7k; MFR (none) -> 4608X-AP1-472LF; Mouser (none) -> 652-4608X-AP1-472LF
- U1: MFR (none) -> SN74LS245N; Mouser (none) -> 595-SN74LS245N
- U10, U11: MFR (none) -> SN74LS74AN; Mouser (none) -> 595-SN74LS74AN
- U12: MFR (none) -> SN74LS244N; Mouser (none) -> 595-SN74LS244N
- U13, U14, U16, U17, U4, U5: MFR (none) -> SN74LS373N; Mouser (none) -> 595-SN74LS373N
- U15, U19: MFR (none) -> ATF16V8B-15PU; Mouser (none) -> 556-AF16V8B15PU
- U2: MFR (none) -> AS6C4008-55PCN; Mouser (none) -> 913-AS6C4008-55PCN
- U3: MFR (none) -> SN74LS75N; Mouser (none) -> 595-SN74LS75N
- U6: MFR (none) -> AT28C64B-15PU; Mouser (none) -> 556-AT28C64B15PU
- U7: MFR (none) -> SN74LS04N; Mouser (none) -> 595-SN74LS04N
- U7: footprint (none) -> Package_DIP:DIP-14_W7.62mm_Socket_LongPads; MFR (none) -> SN74LS04N; Mouser (none) -> 595-SN74LS04N
- U8: MFR (none) -> SN74F08N; Mouser (none) -> 595-SN74F08N
- U9: MFR (none) -> SN74LS21N; Mouser (none) -> 595-SN74LS21N
- Y1: MFR (none) -> HC-49/U-S15000000ABJB; Mouser (none) -> 695-HC49US-15-U
Connections:
- net A10: no longer U6.21 (A10)
- net A11: no longer U6.23 (A11)
- net A8: no longer U6.25 (A8)
- net A9: no longer U6.24 (A9)
- net Q10: now also U6.21 (A10)
- net Q11: now also U6.23 (A11)
- net Q8: now also U6.25 (A8)
- net Q9: now also U6.24 (A9)
- net U2OE: no longer U1.1 (A->B)
- net ~{RD}: now also U1.1 (A->B)

Commit message: kicad: Update titan clone to kicad 9 and add BOM CSV
Parts:
- CN1, U18, U20: now left out of the parts list
- U15: Firmware (none) -> TITAN.JED
- U19: Firmware (none) -> IODECODE.JED
- U6: Firmware (none) -> QXPC.ROM
Connections:
- no-connect marks 45 -> 49
Other:
- moved on the sheet: C1, C11, C13, C15, C17, C19, C21, C22, C3, C5, C7, C9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
